File: hardware/cn3083-breakout/breakout.brd (EAGLE design)
At the start: 23 x 23 mm, 14 parts, among them U1 CN3083

Commit message: added caps for cn3083, oops
Parts:
- removed H3: MOUNT-PAD-ROUND3.0, dtb:3,0-PAD
- added J1: (no value), dtb:JST-2-TH
- moved C2 1.14 mm to (13.0, 4.32), turned to 180 degrees
Connections:
- net GND: now also J1.2
- net VBATT: now also J1.1
Routing:
- net VBATT: track 36.2 -> 43.7 mm
Changed lines of the file:
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@@
 <layer number="23" name="tOrigins" color="15" fill="1" visible="yes" active="yes"/>
 <layer number="24" name="bOrigins" color="15" fill="1" visible="yes" active="yes"/>
-<layer number="25" name="tNames" color="7" fill="1" visible="no" active="yes"/>
+<layer number="25" name="tNames" color="7" fill="1" visible="yes" active="yes"/>
 <layer number="26" name="bNames" color="7" fill="1" visible="no" active="yes"/>
 <layer number="27" name="tValues" color="7" fill="1" visible="no" active="yes"/>
@@
 <text x="14.732" y="0.762" size="1.27" layer="22" font="vector" ratio="14" rot="MR0">APR 15</text>
 <text x="13.97" y="2.54" size="1.27" layer="22" font="vector" ratio="14" rot="MR0">REV A</text>
+<text x="7.112" y="7.366" size="1.524" layer="21" font="vector" ratio="14" rot="R270">BATT</text>
 </plain>
 <attributes>
@@
 <attribute name="NAME" x="9.906" y="21.59" size="1.016" layer="25" font="vector" ratio="14" rot="R180"/>
 </element>
-<element name="C2" library="passives-7351" package="C0603-N" value="4.7u" x="12.446" y="3.302" smashed="yes" rot="R270">
-<attribute name="NAME" x="10.297078125" y="4.35290625" size="1.016" layer="25" font="vector" ratio="14" rot="R270"/>
-</element>
-<element name="H3" library="dtb" package="3,0-PAD" value="MOUNT-PAD-ROUND3.0" x="4.064" y="4.064"/>
+<element name="C2" library="passives-7351" package="C0603-N" value="4.7u" x="12.954" y="4.318" smashed="yes" rot="R180">
+<attribute name="NAME" x="13.49690625" y="3.418921875" size="1.016" layer="25" font="vector" ratio="14" rot="R180"/>
+</element>
+<element name="J1" library="dtb" package="JST-2-TH" value="" x="4.064" y="4.572" rot="R90"/>
 </elements>
 <signals>
@@
 <vertex x="-0.254" y="0"/>
 </polygon>
+<contactref element="J1" pad="2"/>
 </signal>
 <signal name="VBATT">
@@
 <contactref element="R3" pad="1"/>
 <contactref element="C2" pad="1"/>
-<wire x1="14.605" y1="6.223" x2="12.446" y2="6.223" width="0.508" layer="1"/>
-<wire x1="12.446" y1="6.223" x2="11.303" y2="6.223" width="0.508" layer="1"/>
+<wire x1="14.605" y1="6.223" x2="13.716" y2="6.223" width="0.508" layer="1"/>
+<wire x1="13.716" y1="6.223" x2="12.446" y2="6.223" width="0.508" layer="1"/>
+<wire x1="12.446" y1="6.223" x2="11.43" y2="6.223" width="0.508" layer="1"/>
+<wire x1="11.43" y1="6.223" x2="11.303" y2="6.223" width="0.508" layer="1"/>
 <wire x1="9.779" y1="8.83" x2="9.779" y2="7.747" width="0.508" layer="1"/>
 <wire x1="9.779" y1="7.747" x2="11.303" y2="6.223" width="0.508" layer="1"/>
@@
 <wire x1="16.256" y1="15.748" x2="15.748" y2="15.24" width="0.254" layer="1"/>
 <wire x1="15.748" y1="15.24" x2="15.748" y2="10.16" width="0.254" layer="1"/>
-<wire x1="12.446" y1="4.102" x2="12.446" y2="6.223" width="0.254" layer="1"/>
 <wire x1="15.748" y1="10.16" x2="16.256" y2="9.652" width="0.254" layer="1"/>
+<contactref element="J1" pad="1"/>
+<wire x1="13.754" y1="4.318" x2="13.754" y2="6.185" width="0.254" layer="1"/>
+<wire x1="13.754" y1="6.185" x2="13.716" y2="6.223" width="0.254" layer="1"/>
+<wire x1="4.064" y1="5.572" x2="10.779" y2="5.572" width="0.508" layer="1"/>
+<wire x1="10.779" y1="5.572" x2="11.43" y2="6.223" width="0.508" layer="1"/>
 </signal>
 <signal name="N$6">
