File: hardware/cn3083-breakout/breakout.sch (EAGLE design)
At the start: 14 parts, among them U1 CN3083

Commit message: added caps for cn3083, oops
Parts:
- removed H3: MOUNT-PAD-ROUND3.0, dtb:MOUNT-PAD-ROUND3.0
- added J1: (no value), dtb:JST_2MM_MALE_TH
Connections:
- net GND: now also J1.-
- net VBATT: now also J1.+
Changed lines of the file:
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@@
 <part name="GND4" library="SparkFun-Aesthetics" deviceset="GND" device=""/>
 <part name="C2" library="passives-7351" deviceset="CAPACITOR" device="0603-N" value="4.7u"/>
-<part name="H3" library="dtb" deviceset="MOUNT-PAD-ROUND" device="3.0"/>
+<part name="J1" library="dtb" deviceset="JST_2MM_MALE_TH" device=""/>
 </parts>
 <sheets>
@@
 <instance part="GND4" gate="1" x="43.18" y="63.5"/>
 <instance part="C2" gate="G$1" x="137.16" y="71.12"/>
-<instance part="H3" gate="G$1" x="53.34" y="22.86"/>
+<instance part="J1" gate="G$1" x="35.56" y="43.18" rot="R90"/>
 </instances>
 <busses>
@@
 <pinref part="GND4" gate="1" pin="GND"/>
 </segment>
+<segment>
+<pinref part="J1" gate="G$1" pin="-"/>
+<wire x1="40.64" y1="43.18" x2="43.18" y2="43.18" width="0.1524" layer="91"/>
+<label x="43.18" y="43.18" size="1.27" layer="95" xref="yes"/>
+</segment>
 </net>
 <net name="VBATT" class="0">
@@
 <wire x1="137.16" y1="78.74" x2="137.16" y2="73.66" width="0.1524" layer="91"/>
 </segment>
+<segment>
+<pinref part="J1" gate="G$1" pin="+"/>
+<wire x1="40.64" y1="45.72" x2="43.18" y2="45.72" width="0.1524" layer="91"/>
+<label x="43.18" y="45.72" size="1.27" layer="95" xref="yes"/>
+</segment>
 </net>
